Commit message: 2024.02.18调整夹爪姿态使其可以夹住球，封装了一个catch动作作为样例

File: my_robot_controller/urdf/robomasterEP/arm.urdf.xacro (robot description, xacro)
@@ -256,5 +256,5 @@
     </link>
     <joint name="${tf_prefix}arm_1_joint" type="fixed">
-      <origin xyz="0.0103961 -0.0255713 0.030741" rpy="0 0 0"/>
+      <origin xyz="0.0103961 -0.0255713 0.030741" rpy="0 1.3 0"/>
       <parent link="${tf_prefix}arm_base_link"/>
       <child link="${tf_prefix}arm_1_link"/>
@@ -268,5 +268,5 @@
     </joint> -->
     <joint name="${tf_prefix}arm_2_joint" type="fixed">
-      <origin xyz="0.0018704 0.0438659 0.1210238" rpy="0 0 0"/>
+      <origin xyz="0.0018704 0.0438659 0.1210238" rpy="0 -0.5 0"/>
       <parent link="${tf_prefix}arm_1_link"/>
       <child link="${tf_prefix}arm_2_link"/>
@@ -295,5 +295,5 @@
       <child link="${tf_prefix}end_point_link"/>
     </joint>
-    <joint name="${tf_prefix}endpoint_bracket_joint" type="continuous">
+    <joint name="${tf_prefix}endpoint_bracket_joint" type="fixed">
       <origin xyz="0.1058557 0.006752 -0.0561093" rpy="0 0 0"/>
       <parent link="${tf_prefix}arm_2_link"/>
@@ -308,5 +308,5 @@
       <child link="rod_1_dummy"/>
     </joint> -->
-    <joint name="${tf_prefix}rod_1_joint" type="continuous">
+    <joint name="${tf_prefix}rod_1_joint" type="fixed">
       <origin xyz="0.0134583 -0.0540971 0.0213068" rpy="0 -0.021293 0"/>
       <parent link="${tf_prefix}endpoint_bracket_link"/>
@@ -320,6 +320,6 @@
       <child link="rod_2_dummy"/>
     </joint> -->
-    <joint name="${tf_prefix}rod_2_joint" type="continuous">
-      <origin xyz="-0.0224276 -0.0290701 0.0554782" rpy="0 -0.0094248 0"/>
+    <joint name="${tf_prefix}rod_2_joint" type="fixed">
+      <origin xyz="-0.0224276 -0.0290701 0.0554782" rpy="0 1.3 0"/>
       <parent link="${tf_prefix}arm_base_link"/>
       <child link="${tf_prefix}rod_2_link"/>
@@ -333,6 +333,6 @@
       <child link="rod_3_dummy"/>
     </joint> -->
-    <joint name="${tf_prefix}rod_3_joint" type="revolute">
-      <origin xyz="-0.042397 0.0004533 0.0223131" rpy="0 0 0"/>
+    <joint name="${tf_prefix}rod_3_joint" type="fixed">
+      <origin xyz="-0.042397 0.0004533 0.0223131" rpy="0 0.5 0"/>
       <parent link="${tf_prefix}rod_link"/>
       <child link="${tf_prefix}rod_3_link"/>
@@ -340,6 +340,6 @@
       <limit effort="1" velocity="1" lower="-0.34732" upper="1.21475"/>
     </joint>
-    <joint name="${tf_prefix}rod_joint" type="revolute">
-      <origin xyz="0.009805 0.0214241 0.0319234" rpy="0 0 0"/>
+    <joint name="${tf_prefix}rod_joint" type="fixed">
+      <origin xyz="0.009805 0.0214241 0.0319234" rpy="0 0.8 0"/>
       <parent link="${tf_prefix}arm_base_link"/>
       <child link="${tf_prefix}rod_link"/>
@@ -357,6 +357,6 @@
       <child link="triangle_2_dummy"/>
     </joint> -->
-    <joint name="${tf_prefix}triangle_joint" type="continuous">
-      <origin xyz="0.0020224 -0.007103 0.1212334" rpy="0 0.2502802 0"/>
+    <joint name="${tf_prefix}triangle_joint" type="fixed">
+      <origin xyz="0.0020224 -0.007103 0.1212334" rpy="0 -1.1 0"/>
       <parent link="${tf_prefix}arm_1_link"/>
       <child link="${tf_prefix}triangle_link"/>
@@ -382,5 +382,5 @@
         </joint>
     </transmission> -->
-    <transmission name="${tf_prefix}endpoint_bracket_joint">
+    <!-- <transmission name="${tf_prefix}endpoint_bracket_joint">
         <type>transmission_interface/SimpleTransmission</type>
         <actuator name="$${tf_prefix}endpoint_bracket_joint">
@@ -435,5 +435,5 @@
             <hardwareInterface>hardware_interface/VelocityJointInterface</hardwareInterface>
         </joint>
-    </transmission>
+    </transmission> -->
     </xacro:macro>
   </robot>

File: my_robot_controller/urdf/robomasterEP/gripper.urdf.xacro (robot description, xacro)
@@ -152,5 +152,5 @@
       <link name="${tf_prefix}gripper_t_link">
       </link>
-      <joint name="${tf_prefix}gripper_m_joint" type="prismatic">
+      <joint name="${tf_prefix}gripper_m_joint" type="fixed">
         <limit effort="10000" velocity="1" lower="-0.023" upper="0.001"/>
         <origin xyz="0 0 0" rpy="0 0 0"/>
@@ -294,12 +294,12 @@
           </inertial>
         </link> -->
-        <joint name="${tf_prefix}left_gripper_joint_1" type="continuous">
+        <joint name="${tf_prefix}left_gripper_joint_1" type="revolute">
           <origin xyz="0.0163032 0.0212032 -0.0399201" rpy="0 0 0"/>
           <parent link="${tf_prefix}gripper_m_link"/>
           <child link="${tf_prefix}left_gripper_link_1"/>
           <axis xyz="0 0 1.0"/>
-          <limit effort="1" velocity="1"/>
-        </joint>
-        <joint name="${tf_prefix}left_gripper_joint_2" type="continuous">
+          <limit effort="10" velocity="5" lower="-0.4" upper="0"/>
+        </joint>
+        <joint name="${tf_prefix}left_gripper_joint_2" type="fixed">
           <origin xyz="0.0213495 0.0130363 0" rpy="0 0 0"/>
           <parent link="${tf_prefix}left_gripper_link_1"/>
@@ -313,5 +313,5 @@
           <child link="left_gripper_link_3_dummy"/>
         </joint> -->
-        <joint name="${tf_prefix}left_gripper_joint_4" type="continuous">
+        <joint name="${tf_prefix}left_gripper_joint_4" type="fixed">
           <origin xyz="0.00485 0.0204148 -5.8e-06" rpy="0 0 0"/>
           <parent link="${tf_prefix}left_gripper_link_2"/>
@@ -320,5 +320,5 @@
           <limit effort="1" velocity="1"/>
         </joint>
-        <joint name="${tf_prefix}left_gripper_joint_6" type="continuous">
+        <joint name="${tf_prefix}left_gripper_joint_6" type="fixed">
           <origin xyz="0.0051144 -0.0140851 0" rpy="0 0 0"/>
           <parent link="${tf_prefix}left_gripper_link_5"/>
@@ -327,5 +327,5 @@
           <limit effort="1" velocity="1"/>
         </joint>
-        <joint name="${tf_prefix}left_gripper_joint_7" type="continuous">
+        <joint name="${tf_prefix}left_gripper_joint_7" type="fixed">
           <origin xyz="-0.0148823 -0.0168513 0" rpy="0 0 0"/>
           <parent link="${tf_prefix}left_gripper_link_6"/>
@@ -339,5 +339,5 @@
           <child link="left_gripper_8_link_dummy"/>
         </joint> -->
-        <joint name="${tf_prefix}left_gripper_joint_5" type="continuous">
+        <joint name="${tf_prefix}left_gripper_joint_5" type="fixed">
           <origin xyz="0.0385916 0.0103143 1.6e-06" rpy="0 0 0"/>
           <parent link="${tf_prefix}left_gripper_link_4"/>
@@ -347,16 +347,16 @@
         </joint>
         <joint name="${tf_prefix}gripper_joint" type="fixed">
-          <origin xyz="0.0002793 -0.027026 0.0001815" rpy="0 0 0"/>
+          <origin xyz="0.0002793 -0.027026 0.0001815" rpy="0 -0.8 0"/>
           <parent link="${tf_prefix}endpoint_bracket_link"/>
           <child link="${tf_prefix}gripper_link"/>
         </joint>
-        <joint name="${tf_prefix}right_gripper_joint_1" type="continuous">
+        <joint name="${tf_prefix}right_gripper_joint_1" type="revolute">
           <origin xyz="0.0163034 -0.0209781 -0.0399201" rpy="0 0 0"/>
           <parent link="${tf_prefix}gripper_m_link"/>
           <child link="${tf_prefix}right_gripper_link_1"/>
           <axis xyz="0 0 1.0"/>
-          <limit effort="1" velocity="1"/>
-        </joint>
-        <joint name="${tf_prefix}right_gripper_joint_2" type="continuous">
+          <limit effort="10" velocity="5" lower="0" upper="0.4"/>
+        </joint>
+        <joint name="${tf_prefix}right_gripper_joint_2" type="fixed">
           <origin xyz="0.0213495 -0.0130363 0" rpy="0 0 0"/>
           <parent link="${tf_prefix}right_gripper_link_1"/>
@@ -370,5 +370,5 @@
           <child link="right_gripper_link_3_dummy"/>
         </joint> -->
-        <joint name="${tf_prefix}right_gripper_joint_4" type="continuous">
+        <joint name="${tf_prefix}right_gripper_joint_4" type="fixed">
           <origin xyz="0.0047151 -0.0208481 -5.8e-06" rpy="0 0 0"/>
           <parent link="${tf_prefix}right_gripper_link_2"/>
@@ -377,5 +377,5 @@
           <limit effort="1" velocity="1"/>
         </joint>
-        <joint name="${tf_prefix}right_gripper_joint_5" type="continuous">
+        <joint name="${tf_prefix}right_gripper_joint_5" type="fixed">
           <origin xyz="0.0385916 -0.0103143 1.6e-06" rpy="0 0 0"/>
           <parent link="${tf_prefix}right_gripper_link_4"/>
@@ -384,5 +384,5 @@
           <limit effort="1" velocity="1"/>
         </joint>
-        <joint name="${tf_prefix}right_gripper_joint_6" type="continuous">
+        <joint name="${tf_prefix}right_gripper_joint_6" type="fixed">
           <origin xyz="0.0059278 0.0133069 0" rpy="0 0 0"/>
           <parent link="${tf_prefix}right_gripper_link_5"/>
@@ -391,5 +391,5 @@
           <limit effort="1" velocity="1"/>
         </joint>
-        <joint name="${tf_prefix}right_gripper_joint_7" type="continuous">
+        <joint name="${tf_prefix}right_gripper_joint_7" type="fixed">
           <origin xyz="-0.0156955 0.0176295 0" rpy="0 0 0"/>
           <parent link="${tf_prefix}right_gripper_link_6"/>
@@ -398,9 +398,4 @@
           <limit effort="1" velocity="1"/>
         </joint>
-        <!-- <joint name="right_gripper_joint_8_dummy" type="fixed">
-          <origin xyz="-0.0147421 0.0167196 -3.77e-05" rpy="0 0 0"/>
-          <parent link="right_gripper_link_7"/>
-          <child link="right_gripper_link_8_dummy"/>
-        </joint> -->
         <joint name="${tf_prefix}gripper_joint_t" type="fixed">
           <origin xyz="0.124 0 -0.039" rpy="0 0 0"/>
@@ -408,5 +403,5 @@
           <child link="${tf_prefix}gripper_t_link"/>
         </joint>
- <transmission name="${tf_prefix}gripper_m_joint">
+ <!-- <transmission name="${tf_prefix}gripper_m_joint">
         <type>transmission_interface/SimpleTransmission</type>
         <joint name="${tf_prefix}gripper_m_joint">
@@ -417,15 +412,16 @@
             <mechanicalReduction>1</mechanicalReduction>
         </actuator>
-    </transmission>
+    </transmission> -->
     <transmission name="${tf_prefix}left_gripper_joint_1">
         <type>transmission_interface/SimpleTransmission</type>
         <actuator name="$${tf_prefix}left_gripper_joint_1">
+            <hardwareInterface>hardware_interface/EffortJointInterface</hardwareInterface>
             <mechanicalReduction>1</mechanicalReduction>
         </actuator>
         <joint name="${tf_prefix}left_gripper_joint_1">
-            <hardwareInterface>hardware_interface/VelocityJointInterface</hardwareInterface>
-        </joint>
-    </transmission>
-    <transmission name="${tf_prefix}left_gripper_joint_2">
+            <hardwareInterface>hardware_interface/EffortJointInterface</hardwareInterface>
+        </joint>
+    </transmission>
+    <!-- <transmission name="${tf_prefix}left_gripper_joint_2">
         <type>transmission_interface/SimpleTransmission</type>
         <actuator name="$${tf_prefix}left_gripper_joint_2">
@@ -471,15 +467,16 @@
             <hardwareInterface>hardware_interface/VelocityJointInterface</hardwareInterface>
         </joint>
-    </transmission>
+    </transmission> -->
     <transmission name="${tf_prefix}right_gripper_joint_1">
         <type>transmission_interface/SimpleTransmission</type>
         <actuator name="$${tf_prefix}right_gripper_joint_1">
+            <hardwareInterface>hardware_interface/EffortJointInterface</hardwareInterface>
             <mechanicalReduction>1</mechanicalReduction>
         </actuator>
         <joint name="${tf_prefix}right_gripper_joint_1">
-            <hardwareInterface>hardware_interface/VelocityJointInterface</hardwareInterface>
-        </joint>
-    </transmission>
-    <transmission name="${tf_prefix}right_gripper_joint_2">
+            <hardwareInterface>hardware_interface/EffortJointInterface</hardwareInterface>
+        </joint>
+    </transmission>
+    <!-- <transmission name="${tf_prefix}right_gripper_joint_2">
         <type>transmission_interface/SimpleTransmission</type>
         <actuator name="$${tf_prefix}right_gripper_joint_2">
@@ -525,5 +522,5 @@
             <hardwareInterface>hardware_interface/VelocityJointInterface</hardwareInterface>
         </joint>
-    </transmission>
+    </transmission> -->
   </xacro:macro>
 </robot>

File: my_robot_controller/urdf/robomasterEP/wheel.urdf.xacro (robot description, xacro)
@@ -41,5 +41,5 @@
       <limit effort="30" velocity="1.0"/>
     </joint>
-    <transmission name="${name}_wheel_transimission">
+    <!-- <transmission name="${name}_wheel_transimission">
         <type>transmission_interface/SimpleTransmission</type>
         <actuator name="$${name}_motor">
@@ -49,5 +49,5 @@
             <hardwareInterface>hardware_interface/VelocityJointInterface</hardwareInterface>
         </joint>
-    </transmission>
+    </transmission> -->
   </xacro:macro>
 </robot>
