Commit message: 添加了shoot函数，增加了readme中关于移动deepsoccer_gazebo文件夹的提示，实现了catch然后shoot的开环demo

File: my_robot_controller/urdf/robomasterEP/base.urdf.xacro (robot description, xacro)
@@ -8,5 +8,5 @@
       <inertial>
         <origin xyz="-0.0058789 -0.0001128 0.0294307" rpy="0 0 0"/>
-        <mass value="1.934"/>
+        <mass value="9.934"/>
         <inertia ixx="0.01451" ixy="0" ixz="0" iyy="0.00512" iyz="0" izz="0.01759"/>
       </inertial>
